File: grippy/grippy.kicad_sch (KiCad schematic)
At the start: 9 parts, among them J1 Conn_01x08_Socket, SW0 SW_SPST, SW1 SW_SPST, SW2 SW_SPST, SW3 SW_SPST, SW4 SW_SPST, SW5 SW_DPDT_x2, U1 esp32s3-supermini

Commit message: got a board
ready to burn
Connections:
- net B+: now also SW5.2 (B); no longer SW5.1 (A)
- net BLK: now also U1.IO13; no longer U1.IO8
- net CS: now also U1.IO12; no longer U1.IO9
- net DC: now also U1.IO11; no longer U1.IO10
- net RAW: now also SW5.1 (A); no longer SW5.2 (B)
- net RES: now also U1.IO10; no longer U1.IO11
- net SCL: now also U1.IO8; no longer U1.IO13
- net SDA: now also U1.IO9; no longer U1.IO12
Other:
- moved on the sheet: U1

Commit message: repo cleanup / readme started / images
Parts:
- J1: footprint footprints:tft-169-st7789 -> footprints:tft-169-st7789-rt-ang
Changed lines of the file:
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@@
 			)
 		)
-		(property "Footprint" "footprints:tft-169-st7789"
+		(property "Footprint" "footprints:tft-169-st7789-rt-ang"
 			(at 242.57 73.66 0)
 			(effects
